Commit message: camera now points the right way

File: ros2_ws/src/ur5e_rgbd/urdf/ur5e_rgbd.xacro (robot description, xacro)
@@ -19,5 +19,5 @@
     <parent link="wrist_3_link"/>
     <child link="realsense_mount"/>
-    <origin xyz="0 0.02 0.02" rpy="0 0.2 0"/>
+    <origin xyz="0.08 0.0 -0.02" rpy="0 -1.86 0"/>
   </joint>
   <!-- camera -->
