Commit message: fixing camera upside down error

File: ros2_ws/src/ur5e_simulator/urdf/ur5e_rgbd.xacro (robot description, xacro)
@@ -17,7 +17,7 @@
   <link name="realsense_mount"/>
   <joint name="realsense_mount_joint" type="fixed">
-    <parent link="wrist_3_link"/>
+    <parent link="tool0"/>
     <child link="realsense_mount"/>
-    <origin xyz="0.08 0.0 -0.02" rpy="0 -1.86 0"/>
+    <origin xyz="0.08 0.0 -0.02" rpy="${pi} -1.86 0"/>
   </joint>
   <!-- camera -->
@@ -27,4 +27,5 @@
     <!-- Gazebo RGBD sensor -->
   <gazebo reference="realsense_mount">
+    <disableFixedJointLumping>true</disableFixedJointLumping>
     <sensor name="rgbd_camera" type="rgbd_camera">
       <update_rate>30</update_rate>
